Commit message: Complete KUKA iiwa7 action and model integration
Add ROS action/perception intake, trigger-service gripper support, and aligned MoveIt launch assets.

Synchronize calibrated TCP and inertia definitions across planning and simulation, and harden Isaac close validation and timing.

File: ros2_ws/src/robot_integration_ros/urdf/iiwa7_y_gripper_moveit.urdf.xacro (robot description, xacro)
@@ -1,180 +1,194 @@
 <?xml version='1.0' encoding='utf-8'?>
-<robot name="kuka_iiwa7_y_gripper">
-  <link name="base_link">
+<robot xmlns:xacro="http://www.ros.org/wiki/xacro" name="iiwa7">
+  <!-- Generated from assets/urdf/kuka_iiwa7_y_gripper/urdf/kuka_iiwa7_y_gripper.urdf; do not hand-edit. -->
+  <xacro:include filename="$(find lbr_description)/ros2_control/lbr_system_interface.xacro" />
+  <xacro:arg name="robot_name" default="lbr" />
+  <xacro:arg name="mode" default="mock" />
+  <xacro:arg name="system_config_path" default="$(find lbr_description)/ros2_control/lbr_system_config.yaml" />
+  <xacro:arg name="initial_joint_positions_path" default="$(find lbr_description)/ros2_control/initial_joint_positions.yaml" />
+  <xacro:property name="PI" value="3.1415926535897931" />
+  <xacro:property name="joint_limits_path" value="$(find lbr_description)/urdf/iiwa7/joint_limits.yaml" />
+  <xacro:property name="joint_limits" value="${xacro.load_yaml(joint_limits_path)}" />
+  <link name="world" />
+  <joint name="$(arg robot_name)_world_joint" type="fixed">
+    <parent link="world" />
+    <child link="$(arg robot_name)_link_0" />
+  </joint>
+  <link name="$(arg robot_name)_link_0">
     <inertial>
       <origin xyz="-0.0128567641 7.05371085e-07 0.0679655593" rpy="0 0 0" />
       <mass value="30.2763518" />
       <inertia ixx="0.111239566" ixy="-3.81097437e-07" ixz="0.00486659751" iyy="0.139017104" iyz="7.87871532e-07" izz="0.133028622" />
-      </inertial>
-    <visual>
-      <origin xyz="0 0 0" rpy="0 0 0" />
-      <geometry>
-        <mesh filename="../meshes/base_link.STL" scale="1 1 1" />
-        </geometry>
-      <material name="kuka_silver">
-        <color rgba="0.647058823529412 0.619607843137255 0.588235294117647 1" />
-        </material>
-      </visual>
-    <collision>
-      <origin xyz="0 0 0" rpy="0 0 0" />
-      <geometry>
-        <mesh filename="../meshes/base_link.STL" scale="1 1 1" />
-        </geometry>
-      </collision>
-    </link>
-  <link name="link1">
+    </inertial>
+    <visual>
+      <origin xyz="0 0 0" rpy="0 0 0" />
+      <geometry>
+        <mesh filename="package://robot_integration_ros/meshes/base_link.STL" scale="1 1 1" />
+      </geometry>
+      <material name="kuka_silver">
+        <color rgba="0.647058823529412 0.619607843137255 0.588235294117647 1" />
+      </material>
+    </visual>
+    <collision>
+      <origin xyz="0 0 0" rpy="0 0 0" />
+      <geometry>
+        <mesh filename="package://robot_integration_ros/meshes/base_link.STL" scale="1 1 1" />
+      </geometry>
+    </collision>
+  </link>
+  <link name="$(arg robot_name)_link_1">
     <inertial>
       <origin xyz="-4.78790442e-07 -0.0348192059 0.120797868" rpy="0 0 0" />
       <mass value="21.1627406" />
       <inertia ixx="0.133321611" ixy="-5.38303163e-07" ixz="9.16989471e-07" iyy="0.127213841" iyz="0.0236704925" izz="0.0471553201" />
-      </inertial>
+    </inertial>
     <visual>
       <origin xyz="0 0 0.19" rpy="0 0 0" />
       <geometry>
-        <mesh filename="../meshes/link1.STL" scale="1 1 1" />
-        </geometry>
-      <material name="kuka_silver">
-        <color rgba="0.647058823529412 0.619607843137255 0.588235294117647 1" />
-        </material>
-      </visual>
+        <mesh filename="package://robot_integration_ros/meshes/link1.STL" scale="1 1 1" />
+      </geometry>
+      <material name="kuka_silver">
+        <color rgba="0.647058823529412 0.619607843137255 0.588235294117647 1" />
+      </material>
+    </visual>
     <collision>
       <origin xyz="0 0 0.19" rpy="0 0 0" />
       <geometry>
-        <mesh filename="../meshes/link1.STL" scale="1 1 1" />
-        </geometry>
-      </collision>
-    </link>
-  <link name="link2">
+        <mesh filename="package://robot_integration_ros/meshes/link1.STL" scale="1 1 1" />
+      </geometry>
+    </collision>
+  </link>
+  <link name="$(arg robot_name)_link_2">
     <inertial>
       <origin xyz="-5.29061672e-07 0.0392906957 0.0844460685" rpy="0 0 0" />
       <mass value="25.1403147" />
       <inertia ixx="0.197631242" ixy="-3.51963819e-07" ixz="-9.50708464e-08" iyy="0.18755727" iyz="0.0367196702" izz="0.0602720614" />
-      </inertial>
+    </inertial>
     <visual>
       <origin xyz="0 0.0105 -0.0025" rpy="-1.57079633 0 0" />
       <geometry>
-        <mesh filename="../meshes/link2.STL" scale="1 1 1" />
-        </geometry>
-      <material name="kuka_silver">
-        <color rgba="0.647058823529412 0.619607843137255 0.588235294117647 1" />
-        </material>
-      </visual>
+        <mesh filename="package://robot_integration_ros/meshes/link2.STL" scale="1 1 1" />
+      </geometry>
+      <material name="kuka_silver">
+        <color rgba="0.647058823529412 0.619607843137255 0.588235294117647 1" />
+      </material>
+    </visual>
     <collision>
       <origin xyz="0 0.0105 -0.0025" rpy="-1.57079633 0 0" />
       <geometry>
-        <mesh filename="../meshes/link2.STL" scale="1 1 1" />
-        </geometry>
-      </collision>
-    </link>
-  <link name="link3">
+        <mesh filename="package://robot_integration_ros/meshes/link2.STL" scale="1 1 1" />
+      </geometry>
+    </collision>
+  </link>
+  <link name="$(arg robot_name)_link_3">
     <inertial>
       <origin xyz="8.94264666e-07 0.0343188245 0.120097948" rpy="0 0 0" />
       <mass value="21.1627874" />
       <inertia ixx="0.133322418" ixy="-2.72387852e-07" ixz="-2.31579647e-07" iyy="0.127213838" iyz="-0.0236710393" izz="0.0471557501" />
-      </inertial>
+    </inertial>
     <visual>
       <origin xyz="0 0 0.1893" rpy="0 0 0" />
       <geometry>
-        <mesh filename="../meshes/link3.STL" scale="1 1 1" />
-        </geometry>
-      <material name="kuka_silver">
-        <color rgba="0.647058823529412 0.619607843137255 0.588235294117647 1" />
-        </material>
-      </visual>
+        <mesh filename="package://robot_integration_ros/meshes/link3.STL" scale="1 1 1" />
+      </geometry>
+      <material name="kuka_silver">
+        <color rgba="0.647058823529412 0.619607843137255 0.588235294117647 1" />
+      </material>
+    </visual>
     <collision>
       <origin xyz="0 0 0.1893" rpy="0 0 0" />
       <geometry>
-        <mesh filename="../meshes/link3.STL" scale="1 1 1" />
-        </geometry>
-      </collision>
-    </link>
-  <link name="link4">
+        <mesh filename="package://robot_integration_ros/meshes/link3.STL" scale="1 1 1" />
+      </geometry>
+    </collision>
+  </link>
+  <link name="$(arg robot_name)_link_4">
     <inertial>
       <origin xyz="9.93437855e-08 -0.0397907045 0.0837462343" rpy="0 0 0" />
       <mass value="25.140329" />
       <inertia ixx="0.19763084" ixy="-3.24564289e-07" ixz="3.90828878e-07" iyy="0.187556898" iyz="-0.0367195589" izz="0.0602723071" />
-      </inertial>
+    </inertial>
     <visual>
       <origin xyz="0 -0.0105 -0.0032" rpy="-1.57079633 0 0" />
       <geometry>
-        <mesh filename="../meshes/link4.STL" scale="1 1 1" />
-        </geometry>
-      <material name="kuka_silver">
-        <color rgba="0.647058823529412 0.619607843137255 0.588235294117647 1" />
-        </material>
-      </visual>
+        <mesh filename="package://robot_integration_ros/meshes/link4.STL" scale="1 1 1" />
+      </geometry>
+      <material name="kuka_silver">
+        <color rgba="0.647058823529412 0.619607843137255 0.588235294117647 1" />
+      </material>
+    </visual>
     <collision>
       <origin xyz="0 -0.0105 -0.0032" rpy="-1.57079633 0 0" />
       <geometry>
-        <mesh filename="../meshes/link4.STL" scale="1 1 1" />
-        </geometry>
-      </collision>
-    </link>
-  <link name="link5">
+        <mesh filename="package://robot_integration_ros/meshes/link4.STL" scale="1 1 1" />
+      </geometry>
+    </collision>
+  </link>
+  <link name="$(arg robot_name)_link_5">
     <inertial>
       <origin xyz="-1.50596451e-07 -0.0298223596 0.0723663276" rpy="0 0 0" />
       <mass value="9.53466993" />
       <inertia ixx="0.0529038961" ixy="6.86274869e-08" ixz="3.57472027e-07" iyy="0.0444942714" iyz="0.0174914068" izz="0.0239916849" />
-      </inertial>
+    </inertial>
     <visual>
       <origin xyz="0 0 0.1886" rpy="0 0 0" />
       <geometry>
-        <mesh filename="../meshes/link5.STL" scale="1 1 1" />
-        </geometry>
-      <material name="kuka_silver">
-        <color rgba="0.647058823529412 0.619607843137255 0.588235294117647 1" />
-        </material>
-      </visual>
+        <mesh filename="package://robot_integration_ros/meshes/link5.STL" scale="1 1 1" />
+      </geometry>
+      <material name="kuka_silver">
+        <color rgba="0.647058823529412 0.619607843137255 0.588235294117647 1" />
+      </material>
+    </visual>
     <collision>
       <origin xyz="0 0 0.1886" rpy="0 0 0" />
       <geometry>
-        <mesh filename="../meshes/link5.STL" scale="1 1 1" />
-        </geometry>
-      </collision>
-    </link>
-  <link name="link6">
+        <mesh filename="package://robot_integration_ros/meshes/link5.STL" scale="1 1 1" />
+      </geometry>
+    </collision>
+  </link>
+  <link name="$(arg robot_name)_link_6">
     <inertial>
       <origin xyz="3.09820422e-06 0.0710485699 -0.00331157704" rpy="0 0 0" />
       <mass value="14.2007599" />
       <inertia ixx="0.0384515763" ixy="2.19173188e-06" ixz="6.70279498e-08" iyy="0.0368124807" iyz="0.00192249677" izz="0.028001094" />
-      </inertial>
+    </inertial>
     <visual>
       <origin xyz="0 0.0707 -0.0039" rpy="-1.57079633 0 0" />
       <geometry>
-        <mesh filename="../meshes/link6.STL" scale="1 1 1" />
-        </geometry>
-      <material name="kuka_silver">
-        <color rgba="0.647058823529412 0.619607843137255 0.588235294117647 1" />
-        </material>
-      </visual>
+        <mesh filename="package://robot_integration_ros/meshes/link6.STL" scale="1 1 1" />
+      </geometry>
+      <material name="kuka_silver">
+        <color rgba="0.647058823529412 0.619607843137255 0.588235294117647 1" />
+      </material>
+    </visual>
     <collision>
       <origin xyz="0 0.0707 -0.0039" rpy="-1.57079633 0 0" />
       <geometry>
-        <mesh filename="../meshes/link6.STL" scale="1 1 1" />
-        </geometry>
-      </collision>
-    </link>
-  <link name="link7">
+        <mesh filename="package://robot_integration_ros/meshes/link6.STL" scale="1 1 1" />
+      </geometry>
+    </collision>
+  </link>
+  <link name="$(arg robot_name)_link_7">
     <inertial>
       <origin xyz="5.28878934e-07 3.37199922e-07 0.00360718224" rpy="0 0 0" />
       <mass value="2.47156969" />
       <inertia ixx="0.00177365937" ixy="-1.24105214e-07" ixz="-2.95409039e-08" iyy="0.00177328723" iyz="-1.57567641e-08" izz="0.00272748711" />
-      </inertial>
+    </inertial>
     <visual>
       <origin xyz="0 0 0.0311" rpy="0 0 0" />
       <geometry>
-        <mesh filename="../meshes/link7.STL" scale="1 1 1" />
-        </geometry>
-      <material name="kuka_silver">
-        <color rgba="0.647058823529412 0.619607843137255 0.588235294117647 1" />
-        </material>
-      </visual>
+        <mesh filename="package://robot_integration_ros/meshes/link7.STL" scale="1 1 1" />
+      </geometry>
+      <material name="kuka_silver">
+        <color rgba="0.647058823529412 0.619607843137255 0.588235294117647 1" />
+      </material>
+    </visual>
     <collision>
       <origin xyz="0 0 0.0311" rpy="0 0 0" />
       <geometry>
-        <mesh filename="../meshes/link7.STL" scale="1 1 1" />
-        </geometry>
-      </collision>
-    </link>
+        <mesh filename="package://robot_integration_ros/meshes/link7.STL" scale="1 1 1" />
+      </geometry>
+    </collision>
+  </link>
   <link name="gripper_base_link">
     <inertial>
@@ -182,21 +196,21 @@
       <mass value="0.8" />
       <inertia ixx="0.00166886667" ixy="0" ixz="0" iyy="0.00145432361" iyz="0" izz="0.00196999027" />
-      </inertial>
-    <visual>
-      <origin xyz="0 0 0" rpy="0 0 0" />
-      <geometry>
-        <mesh filename="../meshes/hand.STL" scale="0.001 0.001 0.001" />
-        </geometry>
+    </inertial>
+    <visual>
+      <origin xyz="0 0 0" rpy="0 0 0" />
+      <geometry>
+        <mesh filename="package://robot_integration_ros/meshes/hand.STL" scale="0.001 0.001 0.001" />
+      </geometry>
       <material name="gripper_body">
         <color rgba="0.55 0.56 0.58 1" />
-        </material>
-      </visual>
-    <collision>
-      <origin xyz="0 0 0" rpy="0 0 0" />
-      <geometry>
-        <mesh filename="../meshes/hand.STL" scale="0.001 0.001 0.001" />
-        </geometry>
-      </collision>
-    </link>
+      </material>
+    </visual>
+    <collision>
+      <origin xyz="0 0 0" rpy="0 0 0" />
+      <geometry>
+        <mesh filename="package://robot_integration_ros/meshes/hand.STL" scale="0.001 0.001 0.001" />
+      </geometry>
+    </collision>
+  </link>
   <link name="left_finger_link">
     <inertial>
@@ -204,21 +218,21 @@
       <mass value="0.08" />
       <inertia ixx="6.74733326e-05" ixy="0" ixz="0" iyy="5.67733333e-05" iyz="0" izz="3.89133326e-05" />
-      </inertial>
-    <visual>
-      <origin xyz="0 0 0" rpy="0 0 0" />
-      <geometry>
-        <mesh filename="../meshes/left_finger.STL" scale="0.001 0.001 0.001" />
-        </geometry>
+    </inertial>
+    <visual>
+      <origin xyz="0 0 0" rpy="0 0 0" />
+      <geometry>
+        <mesh filename="package://robot_integration_ros/meshes/left_finger.STL" scale="0.001 0.001 0.001" />
+      </geometry>
       <material name="finger_dark">
         <color rgba="0.17 0.2 0.22 1" />
-        </material>
-      </visual>
-    <collision>
-      <origin xyz="0 0 0" rpy="0 0 0" />
-      <geometry>
-        <mesh filename="../meshes/left_finger.STL" scale="0.001 0.001 0.001" />
-        </geometry>
-      </collision>
-    </link>
+      </material>
+    </visual>
+    <collision>
+      <origin xyz="0 0 0" rpy="0 0 0" />
+      <geometry>
+        <mesh filename="package://robot_integration_ros/meshes/left_finger.STL" scale="0.001 0.001 0.001" />
+      </geometry>
+    </collision>
+  </link>
   <link name="right_finger_link">
     <inertial>
@@ -226,21 +240,21 @@
       <mass value="0.08" />
       <inertia ixx="6.74733326e-05" ixy="0" ixz="0" iyy="5.67733333e-05" iyz="0" izz="3.89133326e-05" />
-      </inertial>
-    <visual>
-      <origin xyz="0 0 0" rpy="0 0 0" />
-      <geometry>
-        <mesh filename="../meshes/right_finger.STL" scale="0.001 0.001 0.001" />
-        </geometry>
+    </inertial>
+    <visual>
+      <origin xyz="0 0 0" rpy="0 0 0" />
+      <geometry>
+        <mesh filename="package://robot_integration_ros/meshes/right_finger.STL" scale="0.001 0.001 0.001" />
+      </geometry>
       <material name="finger_dark">
         <color rgba="0.17 0.2 0.22 1" />
-        </material>
-      </visual>
-    <collision>
-      <origin xyz="0 0 0" rpy="0 0 0" />
-      <geometry>
-        <mesh filename="../meshes/right_finger.STL" scale="0.001 0.001 0.001" />
-        </geometry>
-      </collision>
-    </link>
+      </material>
+    </visual>
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