Commit message: Add dual-arm hold and symmetry-aware transition planning

File: assets/urdf/kuka_iiwa7_y_gripper/urdf/kuka_iiwa7_y_gripper.urdf (robot description, URDF)
Before this commit: robot kuka_iiwa7_y_gripper, 12 links, 11 joints
Joints:
- joint gripper_tcp_joint: origin xyz=0 0 0.1505 rpy=0 0 0 -> xyz=0 0 0.1455 rpy=0 0 0

File: ros2_ws/src/robot_integration_ros/urdf/iiwa7_y_gripper_moveit.urdf.xacro (robot description, xacro)
@@ -326,5 +326,5 @@
   </joint>
   <joint name="gripper_tcp_joint" type="fixed">
-    <origin xyz="0 0 0.1505" rpy="0 0 0" />
+    <origin xyz="0 0 0.1455" rpy="0 0 0" />
     <parent link="gripper_base_link" />
     <child link="gripper_tcp" />

Commit message: Improve dual-arm transition planning and recovery

File: assets/urdf/kuka_iiwa7_y_gripper/urdf/kuka_iiwa7_y_gripper.urdf (robot description, URDF)
Before this commit: robot kuka_iiwa7_y_gripper, 12 links, 11 joints
Joints:
- joint gripper_mount_joint: origin xyz=0 0 0.0308 rpy=0 0 0 -> xyz=0 0 0.0308 rpy=0 0 3.14159265
- joint gripper_tcp_joint: origin xyz=0 0 0.1455 rpy=0 0 0 -> xyz=0 0 0.1455 rpy=0 0 3.14159265

File: ros2_ws/src/robot_integration_ros/urdf/dual_iiwa7_y_gripper_moveit.urdf.xacro (robot description, xacro)
@@ -322,10 +322,10 @@
   </joint>
   <joint name="lbr_one_gripper_mount_joint" type="fixed">
-    <origin xyz="0 0 0.0308" rpy="0 0 0" />
+    <origin xyz="0 0 0.0308" rpy="0 0 3.14159265" />
     <parent link="lbr_one_link_7" />
     <child link="lbr_one_gripper_base_link" />
   </joint>
   <joint name="lbr_one_gripper_tcp_joint" type="fixed">
-    <origin xyz="0 0 0.1455" rpy="0 0 0" />
+    <origin xyz="0 0 0.1455" rpy="0 0 3.14159265" />
     <parent link="lbr_one_gripper_base_link" />
     <child link="lbr_one_gripper_tcp" />
@@ -666,10 +666,10 @@
   </joint>
   <joint name="lbr_two_gripper_mount_joint" type="fixed">
-    <origin xyz="0 0 0.0308" rpy="0 0 0" />
+    <origin xyz="0 0 0.0308" rpy="0 0 3.14159265" />
     <parent link="lbr_two_link_7" />
     <child link="lbr_two_gripper_base_link" />
   </joint>
   <joint name="lbr_two_gripper_tcp_joint" type="fixed">
-    <origin xyz="0 0 0.1455" rpy="0 0 0" />
+    <origin xyz="0 0 0.1455" rpy="0 0 3.14159265" />
     <parent link="lbr_two_gripper_base_link" />
     <child link="lbr_two_gripper_tcp" />

File: ros2_ws/src/robot_integration_ros/urdf/iiwa7_y_gripper_moveit.urdf.xacro (robot description, xacro)
@@ -321,10 +321,10 @@
   </joint>
   <joint name="gripper_mount_joint" type="fixed">
-    <origin xyz="0 0 0.0308" rpy="0 0 0" />
+    <origin xyz="0 0 0.0308" rpy="0 0 3.14159265" />
     <parent link="$(arg robot_name)_link_7" />
     <child link="gripper_base_link" />
   </joint>
   <joint name="gripper_tcp_joint" type="fixed">
-    <origin xyz="0 0 0.1455" rpy="0 0 0" />
+    <origin xyz="0 0 0.1455" rpy="0 0 3.14159265" />
     <parent link="gripper_base_link" />
     <child link="gripper_tcp" />
